File: Hardware/SparkFun_Thing_Plus_ESP32-S3.kicad_pcb (KiCad board)
At the start: 4 copper layers, 22.9 x 58.4 mm, 139 parts, among them J1 USB_C_Receptacle, J2 microSD_Friction, J3 JST_2mm_LiPo, J4 Qwiic_RA, SW1 SMD_4.6x2.8mm_h2.5mm, SW2 SMD_4.6x2.8mm_h2.5mm, U1 RT9080-3.3, U10 ThingPlus, U2 DT1042-04SO, U3 ESP32-S3-MINI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

Commit message: initial change to riichi pcb
Parts:
- removed C11, C5: 0.1uF, SparkFun-Capacitor:C_0402_1005Metric
- removed D1: Green, SparkFun-LED:LED_0603_1608Metric_Green
- removed D2, D3: BAT60A, SparkFun-Semiconductor-Standard:SOD-323
- removed D4: Yellow, SparkFun-LED:LED_0603_1608Metric_Yellow
- removed D5: Red, SparkFun-LED:LED_0603_1608Metric_Red
- removed D6: WS2812B, SparkFun-LED:WS2812_2020
- removed FID2, FID3: Fiducial_0.5mm, SparkFun-Aesthetic:Fiducial_0.5mm_Mask1mm
- removed the G*** at (113.0, 118.1)
- removed J2: microSD_Friction, SparkFun-Connector:microSD_Friction_Fit_Common
- removed J4: Qwiic_RA, SparkFun-Connector:JST_SMD_1.0mm-4_RA
- removed JP1, JP3: ~, SparkFun-Jumper:Jumper_2_NC_Trace
- removed R1, R2, R3, R4, R5, R6: 10k, SparkFun-Resistor:R_0402_1005Metric
- removed R12, R15: 2.2k, SparkFun-Resistor:R_0402_1005Metric
- removed R14: 1k, SparkFun-Resistor:R_0402_1005Metric
- removed R7: 330, SparkFun-Resistor:R_0402_1005Metric
- removed R9: 4.7k, SparkFun-Resistor:R_0402_1005Metric
- removed Ref**: Val**, SparkFun-Aesthetic:OSHW_Logo_2.5mm
- removed SW1: SMD_4.6x2.8mm_h2.5mm, SparkFun-Switch:Push_SMD_4.6x2.8mm_h2.5mm
- removed TP1, TP2: 1.0mm, SparkFun-Connector:TestPoint-1.0mm
- removed U10: ThingPlus, SparkFun-Board:ThingPlus
- removed kibuzzard-6569F7FC: G***, kibuzzard-6569F7FC
- removed kibuzzard-656A4896: G***, kibuzzard-656A4896
- removed kibuzzard-65A403E0: G***, kibuzzard-65A403E0
- added X1: 32.768kHz, EasyEDA_Lib:CRYSTAL-SMD_L7.0-W3.2-LS7.5, F.Cu at (110.1, 117.1)
- C4: value 10uF -> 4pF; footprint SparkFun-Capacitor:C_0402_1005Metric -> EasyEDA_Lib:C0402; moved to F.Cu
- C8: value 0.1uF -> 4pF; footprint SparkFun-Capacitor:C_0402_1005Metric -> EasyEDA_Lib:C0402
- J3: value JST_2mm_LiPo -> PH-2AWT; footprint SparkFun-Connector:JST_SMD_2.0mm-2 -> EasyEDA_Lib:CONN-SMD_PH-2AWT
- moved C8 23.7 mm to (111.5, 119.4), turned to 0 degrees
- moved C4 14.4 mm to (108.7, 119.4), turned to 180 degrees
- moved J3 1.43 mm to (106.8, 134.0)
Connections:
- C4 pad 1: 3.3V_P -> GND
- C4 pad 2: GND -> XTAL_32K_P
- C8 pad 1: 3.3V_P -> GND
- C8 pad 2: GND -> XTAL_32K_N
- U3 pad 10: ESP6 -> unconnected-(U3-IOA6-Pad10)
- U3 pad 11: ESP7 -> unconnected-(U3-IOA7-Pad11)
- U3 pad 14: ESP10/A0 -> unconnected-(U3-IOA10-Pad14)
- U3 pad 15: ESP11/PICO -> unconnected-(U3-IOA11-Pad15)
- U3 pad 16: ESP12/SCK -> unconnected-(U3-IOA12-Pad16)
- U3 pad 17: ESP13/POCI -> unconnected-(U3-IOA13-Pad17)
- U3 pad 18: ESP14/A1 -> unconnected-(U3-IOA14-Pad18)
- U3 pad 19: ESP15/A2 -> XTAL_32K_P
- U3 pad 20: ESP16/A3 -> XTAL_32K_N
- U3 pad 21: ESP17/A4 -> unconnected-(U3-IOA17-Pad21)
- U3 pad 22: ESP18/A5 -> unconnected-(U3-IOA18-Pad22)
- U3 pad 25: ESP21 -> unconnected-(U3-IO21-Pad25)
- U3 pad 27: ESP47/SDIO2 -> unconnected-(U3-IO47-Pad27)
- U3 pad 28: ESP33/SDIO3 -> unconnected-(U3-IO33-Pad28)
- U3 pad 29: ESP34/SDIO_CMD -> unconnected-(U3-IO34-Pad29)
- U3 pad 30: ESP48/SDIO_~{DET} -> unconnected-(U3-IO48-Pad30)
- U3 pad 34: ESP38/SDIO_CLK -> unconnected-(U3-IO38-Pad34)
- U3 pad 35: ESP39/SDIO0 -> unconnected-(U3-IO39-Pad35)
- U3 pad 36: ESP40/SDIO1 -> unconnected-(U3-IO40-Pad36)
- U3 pad 37: ESP41/LP_CTL -> unconnected-(U3-IO41-Pad37)
- U3 pad 38: ESP42/FREE -> unconnected-(U3-IO42-Pad38)
- U3 pad 39: ESP43/TXO -> unconnected-(U3-TXD0/IO43-Pad39)
- U3 pad 4: ESP0/STAT -> unconnected-(U3-IO0-Pad4)
- U3 pad 40: ESP44/RXI -> unconnected-(U3-RXD0/IO44-Pad40)
- U3 pad 44: ESP46/LED -> unconnected-(U3-IO46-Pad44)
- U3 pad 5: ESP1 -> unconnected-(U3-IOA1-Pad5)
- U3 pad 6: ESP2 -> unconnected-(U3-IOA2-Pad6)
- U3 pad 8: ESP4 -> unconnected-(U3-IOA4-Pad8)
- U3 pad 9: ESP5 -> unconnected-(U3-IOA5-Pad9)
- U5 pad 1: Net-(D4-K) -> unconnected-(U5-STAT-Pad1)
Routing:
- net 3.3V_P: track 89.0 -> 2.60 mm, vias 10 -> 0
- net ESP40/SDIO1: track 47.4 -> 0.00 mm, vias 1 -> 0
- net ESP0/STAT: track 45.0 -> 0.00 mm, vias 4 -> 0
- net ESP38/SDIO_CLK: track 43.0 -> 0.00 mm, vias 1 -> 0
- net ESP39/SDIO0: track 42.5 -> 0.00 mm, vias 1 -> 0
- net ESP47/SDIO2: track 39.9 -> 0.00 mm, vias 1 -> 0
- net ESP33/SDIO3: track 38.8 -> 0.00 mm, vias 1 -> 0
- net ESP48/SDIO_~{DET}: track 38.7 -> 0.00 mm, vias 1 -> 0
- net ESP34/SDIO_CMD: track 38.7 -> 0.00 mm, vias 1 -> 0
- net VUSB: track 58.1 -> 22.3 mm, vias 4 -> 2
- net ESP10/A0: track 32.4 -> 0.00 mm, vias 2 -> 0
- net 3.3V: track 21.4 -> 50.6 mm, vias 5 -> 1
- net ESP14/A1: track 24.0 -> 0.00 mm
- net Net-(D4-K): track 23.3 -> 0.00 mm, vias 2 -> 0
- net ESP~{RST}: track 55.4 -> 34.4 mm, vias 2 -> 0
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- removed copper zone on In2.Cu, net 3.3V
- removed copper zone on In1.Cu, net GND

Commit message: funktioniert wahrscheinlich erst mal
Parts:
- removed FID1, FID4: Fiducial_0.5mm, SparkFun-Aesthetic:Fiducial_0.5mm_Mask1mm
- removed kibuzzard-656A3526: G***, kibuzzard-656A3526
- removed kibuzzard-656A3552: G***, kibuzzard-656A3552
- removed kibuzzard-656A3559: G***, kibuzzard-656A3559
- removed kibuzzard-656A3560: G***, kibuzzard-656A3560
- removed kibuzzard-656A3567: G***, kibuzzard-656A3567
- removed kibuzzard-656A3591: G***, kibuzzard-656A3591
- removed kibuzzard-656A3598: G***, kibuzzard-656A3598
- removed kibuzzard-656A359E: G***, kibuzzard-656A359E
- removed kibuzzard-656A35A5: G***, kibuzzard-656A35A5
- removed kibuzzard-656A35AD: G***, kibuzzard-656A35AD
- removed kibuzzard-656A35B5: G***, kibuzzard-656A35B5
- removed kibuzzard-656A35BC: G***, kibuzzard-656A35BC
- removed kibuzzard-656A35C4: G***, kibuzzard-656A35C4
- removed kibuzzard-656A361F: G***, kibuzzard-656A361F
- removed kibuzzard-656A3668: G***, kibuzzard-656A3668
- removed kibuzzard-656A367B: G***, kibuzzard-656A367B
- removed kibuzzard-656A3687: G***, kibuzzard-656A3687
- removed kibuzzard-656A368C: G***, kibuzzard-656A368C
- removed kibuzzard-656A3691: G***, kibuzzard-656A3691
- removed kibuzzard-656A36A2: G***, kibuzzard-656A36A2
- removed kibuzzard-656A36A7: G***, kibuzzard-656A36A7
- removed kibuzzard-656A36C2: G***, kibuzzard-656A36C2
- removed kibuzzard-656A3878: G***, kibuzzard-656A3878
- removed kibuzzard-656A3D93: G***, kibuzzard-656A3D93
- removed kibuzzard-656A47C5: G***, kibuzzard-656A47C5
- removed kibuzzard-656A482A: G***, kibuzzard-656A482A
- removed kibuzzard-65A9990D: G***, kibuzzard-65A9990D
- removed kibuzzard-65A99912: G***, kibuzzard-65A99912
- added C11: 0.1uF, Capacitor_SMD:C_0402_1005Metric, F.Cu at (110.8, 124.2)
- added C5: 0.1uF, PCM_SparkFun-Capacitor:C_0402_1005Metric, F.Cu at (119.4, 133.6)
- added R1: 1M, PCM_SparkFun-Resistor:R_0603_1608Metric, F.Cu at (119.2, 135.1)
- added R2: 330k, PCM_SparkFun-Resistor:R_0603_1608Metric, F.Cu at (119.2, 131.8)
- C10, C13: footprint SparkFun-Capacitor:C_0402_1005Metric -> Capacitor_SMD:C_0402_1005Metric
- C4, C8: value 4pF -> 15pF
- U3: footprint SparkFun-RF:ESP32-MINI -> EasyEDA_Lib:WIRELM-SMD_ESP32-S3-WROOM-1
- X1: footprint EasyEDA_Lib:CRYSTAL-SMD_L7.0-W3.2-LS7.5 -> EasyEDA_Lib:FC-135R_L3.2-W1.5
- moved C4 19.9 mm to (100.8, 101.1), turned to -90 degrees
- moved C8 15.8 mm to (100.8, 107.7), turned to 90 degrees
- moved X1 15.3 mm to (101.6, 104.4), turned to -90 degrees
- moved C7 4.56 mm to (100.8, 94.7)
- moved C1 4.49 mm to (100.9, 93.2)
- moved J3 3.30 mm to (103.5, 134.0)
- moved U3 3.25 mm to (114.2, 103.6)
Connections:
- C4 pad 2: XTAL_32K_P -> ESP15/XTAL_32K_P
- C8 pad 2: XTAL_32K_N -> ESP16/XTAL_32K_N
- U3 pad 13: ESP9/SCL -> ESP19/D-
- U3 pad 14: unconnected-(U3-IOA10-Pad14) -> ESP20/D+
- U3 pad 17: unconnected-(U3-IOA13-Pad17) -> ESP9/SCL
- U3 pad 18: unconnected-(U3-IOA14-Pad18) -> ESP10/SPI_CS0
- U3 pad 19: XTAL_32K_P -> ESP11/SPI0_MOSI
- U3 pad 2: GND -> 3.3V
- U3 pad 20: XTAL_32K_N -> ESP12/SPI0_SCK
- U3 pad 21: unconnected-(U3-IOA17-Pad21) -> ESP13/SPI0_MISO
- U3 pad 22: unconnected-(U3-IOA18-Pad22) -> ESP14/BAT_ADC
- U3 pad 23: ESP19/D- -> unconnected-(U3-IO21-Pad23)
- U3 pad 24: ESP20/D+ -> unconnected-(U3-IO47-Pad24)
- U3 pad 26: unconnected-(U3-IO26-Pad26) -> ESP45/Q_EN
- U3 pad 28: unconnected-(U3-IO33-Pad28) -> ESP35/~{ALRT}
- U3 pad 3: 3.3V -> ESP~{RST}
- U3 pad 31: ESP35/~{ALRT} -> unconnected-(U3-IO38-Pad31)
- U3 pad 4: unconnected-(U3-IO0-Pad4) -> ESP4/TOUCH4
- U3 pad 40: unconnected-(U3-RXD0/IO44-Pad40) -> GND
- U3 pad 41: ESP45/Q_EN -> GND
- U3 pad 5: unconnected-(U3-IOA1-Pad5) -> ESP5/TOUCH5
- U3 pad 6: unconnected-(U3-IOA2-Pad6) -> ESP6/TOUCH6
- U3 pad 7: unconnected-(U3-IOA3-Pad7) -> ESP7/TOUCH7
- U3 pad 8: unconnected-(U3-IOA4-Pad8) -> ESP15/XTAL_32K_P
- U3 pad 9: unconnected-(U3-IOA5-Pad9) -> ESP16/XTAL_32K_N
- X1 pad 1: XTAL_32K_P -> ESP15/XTAL_32K_P
- X1 pad 2: XTAL_32K_N -> ESP16/XTAL_32K_N
Routing:
- net GND: track 87.9 -> 17.0 mm, vias 53 -> 12
- net ESP14/BAT_ADC: track 0.00 -> 24.5 mm, vias 0 -> 2
- net ESP45/Q_EN: track 61.1 -> 47.9 mm
- net 3.3V: track 50.6 -> 62.4 mm
- net ESP20/D+: track 40.2 -> 48.0 mm
- net XTAL_32K_N: track 7.48 -> 0.00 mm
- net ESP8/SDA: track 60.4 -> 67.3 mm
- net XTAL_32K_P: track 6.95 -> 0.00 mm
- net ESP19/D-: track 41.2 -> 48.1 mm
- net ESP16/XTAL_32K_N: track 0.00 -> 5.97 mm
- net ESP15/XTAL_32K_P: track 0.00 -> 5.88 mm
- net ESP~{RST}: track 34.4 -> 39.4 mm, vias 0 -> 2
- net VBATT: track 22.2 -> 25.2 mm
- net ESP9/SCL: track 58.7 -> 57.4 mm
- net ESP35/~{ALRT}: track 33.5 -> 34.4 mm
Other:
- board size 22.9 x 58.4 mm -> 26.9 x 62 mm
- copper layers 4 -> 2

Commit message: temp
Parts:
- removed G***: LOGO, SparkFun-Aesthetic:SparkFun_Logo_12.5mm
- removed J1: USB_C_Receptacle, SparkFun-Connector:USB-C_16
- removed kibuzzard-6569BE28: G***, kibuzzard-6569BE28
- removed kibuzzard-6569BE4A: G***, kibuzzard-6569BE4A
- removed kibuzzard-6569BE57: G***, kibuzzard-6569BE57
- removed kibuzzard-6569BF02: G***, kibuzzard-6569BF02
- removed kibuzzard-6569F8A4: G***, kibuzzard-6569F8A4
- removed kibuzzard-656A31AF: G***, kibuzzard-656A31AF
- removed kibuzzard-656A32A0: G***, kibuzzard-656A32A0
- removed kibuzzard-656A32FE: G***, kibuzzard-656A32FE
- removed kibuzzard-65A9923A: G***, kibuzzard-65A9923A
- removed kibuzzard-65A99252: G***, kibuzzard-65A99252
- removed kibuzzard-65A99268: G***, kibuzzard-65A99268
- removed kibuzzard-65A9926C: G***, kibuzzard-65A9926C
- removed kibuzzard-65A9926F: G***, kibuzzard-65A9926F
- removed kibuzzard-65A99274: G***, kibuzzard-65A99274
- removed kibuzzard-65A99278: G***, kibuzzard-65A99278
- removed kibuzzard-65A9927C: G***, kibuzzard-65A9927C
- removed kibuzzard-65A9927F: G***, kibuzzard-65A9927F
- removed kibuzzard-65A99283: G***, kibuzzard-65A99283
- removed kibuzzard-65A99287: G***, kibuzzard-65A99287
- removed kibuzzard-65A9928A: G***, kibuzzard-65A9928A
- removed kibuzzard-65A9928E: G***, kibuzzard-65A9928E
- removed kibuzzard-65A99292: G***, kibuzzard-65A99292
- removed kibuzzard-65A99297: G***, kibuzzard-65A99297
- removed kibuzzard-65A992E3: G***, kibuzzard-65A992E3
- removed kibuzzard-65A99335: G***, kibuzzard-65A99335
- removed kibuzzard-65A9933C: G***, kibuzzard-65A9933C
- removed kibuzzard-65A99346: G***, kibuzzard-65A99346
- removed kibuzzard-65A9934B: G***, kibuzzard-65A9934B
- removed kibuzzard-65A99350: G***, kibuzzard-65A99350
- removed kibuzzard-65A99354: G***, kibuzzard-65A99354
- removed kibuzzard-65A99359: G***, kibuzzard-65A99359
- removed kibuzzard-65A9935C: G***, kibuzzard-65A9935C
- removed kibuzzard-65A99360: G***, kibuzzard-65A99360
- removed kibuzzard-65A99364: G***, kibuzzard-65A99364
- removed kibuzzard-65A99367: G***, kibuzzard-65A99367
- removed kibuzzard-65A9936B: G***, kibuzzard-65A9936B
- removed kibuzzard-65A99933: G***, kibuzzard-65A99933
- removed kibuzzard-65A99E72: G***, kibuzzard-65A99E72
- added C15: 1.0uF, Capacitor_SMD:C_0402_1005Metric, F.Cu at (118.3, 130.3)
- added R3: 10k, Resistor_SMD:R_0402_1005Metric, F.Cu at (108.7, 131.1)
- added SW1: C528967, EasyEDA_Lib:SW-SMD_4P-L5.1-W5.1-P3.70-LS6.5-TL_H1.5, F.Cu at (113.8, 131.8)
- added USB2: C2927038, EasyEDA_Lib:USB-C_SMD-TYPE-C-31-M-12, F.Cu at (113.0, 148.9)
- C1: footprint SparkFun-Capacitor:C_0603_1608Metric -> Capacitor_SMD:C_0603_1608Metric
- C12, C14, C3: footprint SparkFun-Capacitor:C_0402_1005Metric -> PCM_SparkFun-Capacitor:C_0402_1005Metric
- C2, C6, C7: footprint SparkFun-Capacitor:C_0402_1005Metric -> Capacitor_SMD:C_0402_1005Metric
- C9: footprint SparkFun-Capacitor:C_0603_1608Metric -> Capacitor_SMD:C_0402_1005Metric
- JP2: footprint SparkFun-Jumper:Jumper_2_NC_Trace -> Jumper:SolderJumper-2_P1.3mm_Bridged_RoundedPad1.0x1.5mm
- R10, R11, R13, R16, R17, R19, R8: footprint SparkFun-Resistor:R_0402_1005Metric -> Resistor_SMD:R_0402_1005Metric
- SW2: value SMD_4.6x2.8mm_h2.5mm -> C528967; footprint SparkFun-Switch:Push_SMD_4.6x2.8mm_h2.5mm -> EasyEDA_Lib:SW-SMD_4P-L5.1-W5.1-P3.70-LS6.5-TL_H1.5
- U1, U6: footprint SparkFun-Semiconductor-Standard:SOT23-5 -> Package_TO_SOT_SMD:SOT-23-5
- U2: footprint SparkFun-Semiconductor-Standard:SOT23-6 -> EasyEDA_Lib:SOT-23-6_L2.9-W1.6-P0.95-LS2.9-BL
- U5: footprint SparkFun-Semiconductor-Standard:SOT23-5 -> EasyEDA_Lib:SOT-23-5_L3.0-W1.7-P0.95-LS2.8-BR
- X1: value 32.768kHz -> C32346
- moved C6 4.35 mm to (120.4, 122.7)
- moved R8 4.24 mm to (121.4, 122.7)
- moved SW2 2.62 mm to (115.8, 124.2)
- moved JP2 1.14 mm to (116.3, 127.1)
- moved U1 0.45 mm to (111.1, 142.4)
- moved C9 0.16 mm to (113.0, 137.6)
- turned U2 to 90 degrees
- turned U5 to 0 degrees
Connections:
- SW2 pad 2: GND -> ESP~{RST}
- U3 pad 27: unconnected-(U3-IO0-Pad27) -> ESP0/BOOT
Routing:
- net ESP0/BOOT: track 0.00 -> 30.5 mm
- net 3.3V: track 62.4 -> 72.7 mm
- net GND: track 17.0 -> 11.7 mm, vias 12 -> 13
- net ESP~{RST}: track 39.4 -> 37.3 mm
- net ESP19/D-: track 48.1 -> 48.9 mm
- net 3.3V_P: track 2.60 -> 1.83 mm
Other:
- board text removed: "v10"

Commit message: update schematic (hopefully final)
Parts:
- SW1, SW2: value C528967 -> C318884
- U1, U6: value RT9080-3.3 -> RT9080-33
Other:
- board size 26.9 x 62 mm -> 123.7 x 123.7 mm
- board text removed: "Controlled Impedance: JLC7628"
- board text removed: "Finish: HASL Lead-Free"
- board text removed: "Layers: 4"
- board text removed: "Material: TG155"
- board text removed: "Solder Mask: Red"
- board text removed: "Thickness: 1.6mm"

Commit message: .
Parts:
- removed C10: 2.2uF, Capacitor_SMD:C_0402_1005Metric
- removed C11: 0.1uF, Capacitor_SMD:C_0402_1005Metric
- removed C12: 4.7uF, PCM_SparkFun-Capacitor:C_0402_1005Metric
- removed G3: OSHW_Logo, SparkFun-Aesthetic:Creative_Commons_License
- removed R17: 10k, Resistor_SMD:R_0402_1005Metric
- removed R19: 100k, Resistor_SMD:R_0402_1005Metric
- removed U5: MCP73831, EasyEDA_Lib:SOT-23-5_L3.0-W1.7-P0.95-LS2.8-BR
- removed U6: RT9080-33, Package_TO_SOT_SMD:SOT-23-5
- added C14: 1uF, Capacitor_SMD:C_0402_1005Metric, F.Cu at (132.3, 145.8)
- added C16: 10uF, PCM_SparkFun-Capacitor:C_0402_1005Metric, F.Cu at (150.6, 144.8)
- added C3: 1uF, Capacitor_SMD:C_0402_1005Metric, F.Cu at (136.1, 150.1)
- added D2: C8678, EasyEDA_Lib:SMA_L4.3-W2.6-LS5.2-RD, F.Cu at (138.3, 147.1)
- added DISP1: Conn_02x04_Counter_Clockwise, Connector_PinSocket_2.54mm:PinSocket_2x04_P2.54mm_Vertical, F.Cu at (135.9, 135.9)
- added J1: PH-2AWT, EasyEDA_Lib:CONN-SMD_PH-2AWT, F.Cu at (103.5, 133.8)
- added J2: Touch1, Connector_PinSocket_2.54mm:PinSocket_1x01_P2.54mm_Horizontal, F.Cu at (82.4, 36.9)
- added J4: Touch3, Connector_PinSocket_2.54mm:PinSocket_1x01_P2.54mm_Horizontal, F.Cu at (151.3, 135.6)
- added J5: Touch4, Connector_PinSocket_2.54mm:PinSocket_1x01_P2.54mm_Horizontal, F.Cu at (56.9, 122.6)
- added LED1: C2297, EasyEDA_Lib:LED0805-R-RD, F.Cu at (110.3, 38.4)
- added LED2: C2297, EasyEDA_Lib:LED0805-R-RD, F.Cu at (166.1, 86.6)
- added LED3: C2297, EasyEDA_Lib:LED0805-R-RD, F.Cu at (102.3, 149.6)
- added LED4: C2297, EasyEDA_Lib:LED0805-R-RD, F.Cu at (57.9, 93.0)
- added Q1: C10487, EasyEDA_Lib:SOT-23-3_L3.0-W1.7-P0.95-LS2.9-BR, F.Cu at (138.6, 142.7)
- added R12: 49.9, Resistor_SMD:R_0402_1005Metric, F.Cu at (125.7, 102.9)
- added R14: 10k, Resistor_SMD:R_0402_1005Metric, F.Cu at (126.2, 91.4)
- added R15: 10k, Resistor_SMD:R_0402_1005Metric, F.Cu at (126.0, 92.7)
- added R16: 10k, Resistor_SMD:R_0402_1005Metric, F.Cu at (126.0, 94.5)
- added R4: 2.0k, Resistor_SMD:R_0402_1005Metric, F.Cu at (145.3, 150.9)
- added R5: 49.9, Resistor_SMD:R_0402_1005Metric, F.Cu at (126.0, 98.8)
- added R6: 100k, Resistor_SMD:R_0402_1005Metric, F.Cu at (138.9, 150.1)
- added R7: 49.9, Resistor_SMD:R_0402_1005Metric, F.Cu at (126.0, 100.8)
- added R9: 49.9, Resistor_SMD:R_0402_1005Metric, F.Cu at (126.0, 96.8)
- added SW3: C318884, EasyEDA_Lib:SW-SMD_4P-L5.1-W5.1-P3.70-LS6.5-TL_H1.5, F.Cu at (63.5, 38.2)
- added SW4: C318884, EasyEDA_Lib:SW-SMD_4P-L5.1-W5.1-P3.70-LS6.5-TL_H1.5, F.Cu at (161.2, 39.2)
- added SW5: C318884, EasyEDA_Lib:SW-SMD_4P-L5.1-W5.1-P3.70-LS6.5-TL_H1.5, F.Cu at (161.8, 141.7)
- added SW6: C318884, EasyEDA_Lib:SW-SMD_4P-L5.1-W5.1-P3.70-LS6.5-TL_H1.5, F.Cu at (63.8, 140.7)
- added U8: C235316, EasyEDA_Lib:SOT-353_L2.1-W1.3-P0.65-LS2.3-BL, F.Cu at (132.3, 148.6)
- C13: value 1.0uF -> 10uF; footprint Capacitor_SMD:C_0402_1005Metric -> PCM_SparkFun-Capacitor:C_0402_1005Metric
- J3: value PH-2AWT -> Touch2; footprint EasyEDA_Lib:CONN-SMD_PH-2AWT -> Connector_PinSocket_2.54mm:PinSocket_1x01_P2.54mm_Horizontal
- R13: value 100k -> 10k
- U1: value RT9080-33 -> C16581; footprint Package_TO_SOT_SMD:SOT-23-5 -> EasyEDA_Lib:ESOP-8_L4.9-W3.9-P1.27-LS6.0-BL-EP
- U2: value DT1042-04SO -> C85364
- moved J3 96.4 mm to (164.8, 59.5), turned to -90 degrees
- moved U3 49.6 mm to (82.8, 142.1)
- moved C13 44.9 mm to (150.6, 147.1), turned to 90 degrees
- moved R13 43.0 mm to (126.0, 90.2), turned to 0 degrees
- moved U1 35.8 mm to (146.7, 146.0), turned to 0 degrees
- moved C15 31.1 mm to (146.2, 116.7)
- moved R3 31.1 mm to (136.6, 117.4)
- moved SW1 31.1 mm to (141.7, 118.1)
- moved C6 29.0 mm to (145.4, 108.0)
- moved SW2 29.0 mm to (140.8, 109.5)
- moved R8 29.0 mm to (146.4, 108.0)
- moved ST3 27.4 mm to (145.3, 164.1)
- moved ST1 25.2 mm to (84.1, 165.1)
- moved U4 11.6 mm to (132.6, 142.9)
- moved C2 11.4 mm to (134.4, 140.7), turned to 180 degrees
Connections:
- C13 pad 1: 3.3V -> VUSB
- J3 pad 1: GND -> ESP5/TOUCH5
- R13 pad 1: VIN -> 3.3V
- R13 pad 2: EN -> ESP39/BUTTON1
- U1 pad 1: VIN -> GND
- U1 pad 2: GND -> Net-(U1-PROG)
- U1 pad 3: ESP45/Q_EN -> GND
- U1 pad 4: unconnected-(U1-NC-Pad4) -> VUSB
- U1 pad 5: 3.3V_P -> VBATT
- U3 pad 10: unconnected-(U3-IO17-Pad10) -> ESP17/DC
- U3 pad 23: unconnected-(U3-IO21-Pad23) -> ESP21/~{ALRT}
- U3 pad 28: ESP35/~{ALRT} -> ESP35/LED1
- U3 pad 29: unconnected-(U3-IO36-Pad29) -> ESP36/LED2
- U3 pad 30: unconnected-(U3-IO37-Pad30) -> ESP37/LED3
- U3 pad 31: unconnected-(U3-IO38-Pad31) -> ESP38/LED4
- U3 pad 32: unconnected-(U3-IO39-Pad32) -> ESP39/BUTTON1
- U3 pad 33: unconnected-(U3-IO40-Pad33) -> ESP40/BUTTON2
- U3 pad 34: unconnected-(U3-IO41-Pad34) -> ESP41/BUTTON3
- U3 pad 35: unconnected-(U3-IO42-Pad35) -> ESP42/BUTTON4
- U3 pad 38: unconnected-(U3-IO2-Pad38) -> ESP2/RES
- U3 pad 39: unconnected-(U3-IO1-Pad39) -> ESP1/BUSY
- U4 pad 5: ESP35/~{ALRT} -> ESP21/~{ALRT}
Routing:
- net VUSB: track 21.9 -> 60.4 mm
- net ESP35/~{ALRT}: track 34.4 -> 0.00 mm, vias 2 -> 0
- net ESP21/~{ALRT}: track 0.00 -> 33.3 mm, vias 0 -> 2
- net VBATT: track 25.2 -> 44.1 mm
- net Net-(D2-K): track 0.00 -> 12.4 mm
- net 3.3V: track 72.7 -> 68.3 mm
- net Net-(U1-PROG): track 0.00 -> 2.09 mm
Other:
- outline, holes or cut-outs redrawn
- board text removed: "N. Seidle"

Commit message: power part done
Parts:
- removed the C14 at (112.1, 144.8)
- removed the C3 at (108.3, 142.9)
- removed JP2: ~, Jumper:SolderJumper-2_P1.3mm_Bridged_RoundedPad1.0x1.5mm
- removed the R16 at (116.5, 140.3)
- removed U9: ~, SparkFun-Aesthetic:Ordering_Instructions
- removed kibuzzard-65A99A9C: G***, kibuzzard-65A99A9C
- removed kibuzzard-65A99AA3: G***, kibuzzard-65A99AA3
- moved C7 43.2 mm to (74.6, 129.0)
- moved C1 43.2 mm to (74.6, 127.5)
- moved C4 41.4 mm to (73.9, 132.5)
- moved C8 41.4 mm to (73.9, 139.2)
- moved X1 41.4 mm to (74.7, 135.9)
- moved J1 39.5 mm to (142.9, 136.9), turned to -90 degrees
- moved DISP1 28.7 mm to (108.3, 128.0)
- moved C9 18.1 mm to (128.2, 147.5), turned to -90 degrees
- moved R2 16.0 mm to (134.0, 125.8)
- moved R1 16.0 mm to (134.0, 129.1)
- moved C5 16.0 mm to (134.2, 127.6)
- moved LED3 9.77 mm to (112.0, 148.3)
- moved U3 9.69 mm to (89.5, 135.1)
- moved R11 8.06 mm to (115.4, 147.6)
- moved U2 8.06 mm to (124.6, 142.8)
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Routing:
- net ESP8/SDA: track 67.3 -> 0.00 mm, vias 4 -> 0
- net ESP9/SCL: track 57.4 -> 0.00 mm, vias 2 -> 0
- net 3.3V: track 68.3 -> 13.4 mm, vias 1 -> 0
- net ESP45/Q_EN: track 48.2 -> 0.00 mm, vias 2 -> 0
- net ESP20/D+: track 47.9 -> 6.77 mm, vias 2 -> 1
- net ESP19/D-: track 48.9 -> 9.35 mm, vias 2 -> 1
- net VIN: track 38.5 -> 0.00 mm, vias 3 -> 0
- net ESP~{RST}: track 37.3 -> 0.00 mm, vias 2 -> 0
- net ESP21/~{ALRT}: track 33.3 -> 0.00 mm, vias 2 -> 0
- net ESP0/BOOT: track 30.5 -> 0.00 mm
- net ESP14/BAT_ADC: track 24.5 -> 4.98 mm, vias 2 -> 0
- net Net-(JP2-A): track 18.0 -> 0.00 mm, vias 3 -> 0
- net VUSB: track 60.4 -> 75.7 mm
- net GND: track 11.7 -> 0.00 mm, vias 13 -> 0
- net VBATT: track 44.1 -> 38.0 mm
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Other:
- outline, holes or cut-outs redrawn
