File: Hardware/SparkFun_Thing_Plus_ESP32-S3.kicad_pcb (KiCad board)
At the start: 2 copper layers, 123.7 x 123.7 mm, 57 parts, among them J1 PH-2AWT, J2 Touch1, J3 Touch2, J4 Touch3, J5 Touch4, Q1 C10487, SW1 C318884, SW2 C318884, SW3 C318884, SW4 C318884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

Commit message: 1st production version
Parts:
- removed R13, R14, R15, R16, R3: 10k, Resistor_SMD:R_0402_1005Metric
- removed ST1, ST3: Standoff, SparkFun-Hardware:Standoff
- removed kibuzzard-65AA9C9F: G***, kibuzzard-65AA9C9F
- added H1: MountingHole, MountingHole:MountingHole_6.4mm_M6_DIN965, F.Cu at (68.9, 130.0)
- added H2: MountingHole, MountingHole:MountingHole_6.4mm_M6_DIN965, F.Cu at (155.1, 130.0)
- added H3: MountingHole, MountingHole:MountingHole_2.7mm_M2.5_ISO14580, F.Cu at (168.3, 116.1)
- added H4: MountingHole, MountingHole:MountingHole_2.7mm_M2.5_ISO14580, F.Cu at (168.3, 66.4)
- added H5: MountingHole, MountingHole:MountingHole_2.7mm_M2.5_ISO14580, F.Cu at (55.7, 66.5)
- added H6: MountingHole, MountingHole:MountingHole_2.7mm_M2.5_ISO14580, F.Cu at (55.7, 116.1)
- moved C6 84.1 mm to (68.8, 142.8), turned to 90 degrees
- moved R8 83.4 mm to (70.6, 142.8), turned to 180 degrees
- moved Reset1 79.4 mm to (71.2, 147.8)
- moved R5 48.1 mm to (103.9, 141.5)
- moved R9 47.6 mm to (103.9, 138.9)
- moved C15 46.6 mm to (109.0, 144.7)
- moved BOOT1 46.5 mm to (104.3, 145.7)
- moved R7 45.2 mm to (103.9, 140.2)
- moved R12 41.1 mm to (103.9, 137.7)
- moved J2 36.9 mm to (54.9, 61.5), turned to -90 degrees
- moved J4 19.2 mm to (169.4, 121.2), turned to 90 degrees
- moved R2 12.9 mm to (130.8, 138.3), turned to 90 degrees
- moved C7 11.4 mm to (71.5, 140.0), turned to -90 degrees
- moved C5 10.7 mm to (132.6, 138.2), turned to -90 degrees
- moved C1 10.5 mm to (71.4, 137.5), turned to -90 degrees
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- renumbered SW1 to BOOT1, SW2 to Reset1
Routing:
- net Net-(LED1-A): track 0.00 -> 198.8 mm, vias 0 -> 2
- net ESP40/BUTTON2: track 0.00 -> 175.1 mm, vias 0 -> 2
- net ESP5/TOUCH5: track 0.00 -> 150.1 mm, vias 0 -> 2
- net ESP39/BUTTON1: track 0.00 -> 129.3 mm, vias 0 -> 2
- net Net-(LED2-A): track 0.00 -> 121.9 mm, vias 0 -> 2
- net 3.3V: track 13.4 -> 125.4 mm
- net ESP6/TOUCH6: track 0.00 -> 96.4 mm, vias 0 -> 2
- net ESP4/TOUCH4: track 0.00 -> 88.1 mm, vias 0 -> 2
- net Net-(LED4-A): track 0.00 -> 84.6 mm, vias 0 -> 2
- net ESP41/BUTTON3: track 0.00 -> 71.1 mm, vias 0 -> 2
- net ESP19/D-: track 9.35 -> 78.1 mm, vias 1 -> 2
- net ESP20/D+: track 6.77 -> 73.7 mm, vias 1 -> 4
- net ESP8/SDA: track 0.00 -> 61.1 mm, vias 0 -> 2
- net ESP17/DC: track 0.00 -> 54.9 mm, vias 0 -> 2
- net ESP9/SCL: track 0.00 -> 52.4 mm, vias 0 -> 2
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Other:
- board size 123.7 x 123.7 mm -> 123.4 x 123.4 mm
