File: Hardware/SparkFun_Thing_Plus_ESP32-S3.kicad_sch (KiCad schematic)
At the start: 35 parts, among them J1 USB_C_Receptacle, SW1 SMD_4.6x2.8mm_h2.5mm, SW2 SMD_4.6x2.8mm_h2.5mm, U10 ThingPlus, U2 DT1042-04SO, U3 ESP32-S3-MINI, U6 RT9080-3.3

Commit message: initial change to riichi pcb
Parts:
- removed D1: Green, SparkFun-LED:LED_0603_1608Metric_Green, symbol SparkFun-LED:LED_Green_0603
- removed D2, D3: BAT60A, SparkFun-Semiconductor-Standard:SOD-323, symbol SparkFun-DiscreteSemi:D_Schottky_3A_10V_0.28V
- removed D5: Red, SparkFun-LED:LED_0603_1608Metric_Red, symbol SparkFun-LED:LED_Red_0603
- removed JP1: ~, SparkFun-Jumper:Jumper_2_NC_Trace, symbol SparkFun-Jumper:SolderJumper_2_Bridged
- removed R7: 330, SparkFun-Resistor:R_0402_1005Metric, symbol SparkFun-Resistor:330_0402
- removed R9: 4.7k, SparkFun-Resistor:R_0402_1005Metric, symbol SparkFun-Resistor:4.7k_0402
- removed SW2: SMD_4.6x2.8mm_h2.5mm, SparkFun-Switch:Push_SMD_4.6x2.8mm_h2.5mm, symbol SparkFun-Switch:SPST_Push_SMD_4.6x2.8mm_h2.5mm
- removed TP2: 1.0mm, SparkFun-Connector:TestPoint-1.0mm, symbol SparkFun-Connector:TestPoint_1.0mm
- removed U10: ThingPlus, SparkFun-Board:ThingPlus, symbol SparkFun-Board:ThingPlus
- renumbered C3 to C6, G3 to G1, R1 to R8, SW1 to SW2
Connections:
- net ESP0/STAT: no longer names the net of U3.4 (IO0)
- net ESP1: no longer names the net of U3.5 (IOA1)
- net ESP10/A0: no longer names the net of U3.14 (IOA10)
- net ESP11/PICO: no longer names the net of U3.15 (IOA11)
- net ESP12/SCK: no longer names the net of U3.16 (IOA12)
- net ESP13/POCI: no longer names the net of U3.17 (IOA13)
- net ESP14/A1: no longer names the net of U3.18 (IOA14)
- net ESP15/A2 renamed XTAL_32K_P
- net ESP16/A3 renamed XTAL_32K_N
- net ESP17/A4: no longer names the net of U3.21 (IOA17)
- net ESP18/A5: no longer names the net of U3.22 (IOA18)
- net ESP2: no longer names the net of U3.6 (IOA2)
- net ESP21: no longer names the net of U3.25 (IO21)
- net ESP33/SDIO3: no longer names the net of U3.28 (IO33)
- net ESP34/SDIO_CMD: no longer names the net of U3.29 (IO34)
- net ESP38/SDIO_CLK: no longer names the net of U3.34 (IO38)
- net ESP39/SDIO0: no longer names the net of U3.35 (IO39)
- net ESP4: no longer names the net of U3.8 (IOA4)
- net ESP40/SDIO1: no longer names the net of U3.36 (IO40)
- net ESP41/LP_CTL: no longer names the net of U3.37 (IO41)
- net ESP42/FREE: no longer names the net of U3.38 (IO42)
- net ESP43/TXO: no longer names the net of U3.39 (TXD0/IO43)
- net ESP44/RXI: no longer names the net of U3.40 (RXD0/IO44)
- net ESP46/LED: no longer names the net of U3.44 (IO46)
- net ESP47/SDIO2: no longer names the net of U3.27 (IO47)
- net ESP48/SDIO_~{DET}: no longer names the net of U3.30 (IO48)
- net ESP5: no longer names the net of U3.9 (IOA5)
- net ESP6: no longer names the net of U3.10 (IOA6)
- net ESP7: no longer names the net of U3.11 (IOA7)

Commit message: funktioniert wahrscheinlich erst mal
Parts:
- removed FID1, FID2, FID3, FID4: Fiducial_0.5mm, SparkFun-Aesthetic:Fiducial_0.5mm_Mask1mm, symbol SparkFun-Aesthetic:Fiducial_0.5mm
- C10, C11, C13: footprint SparkFun-Capacitor:C_0402_1005Metric -> Capacitor_SMD:C_0402_1005Metric
- ST1, ST3: now not fitted
- U3: footprint SparkFun-RF:ESP32-MINI -> EasyEDA_Lib:WIRELM-SMD_ESP32-S3-WROOM-1; symbol SparkFun-RF:ESP32-S3-MINI -> EasyEDA_Lib:ESP32-S3-WROOM-1; LCSC Part Name (none) -> ESP32-S3-WROOM-1; Manufacturer Part (none) -> ESP32-S3-WROOM-1; Supplier (none) -> LCSC; Supplier Part (none) -> C9900163599
Connections:
- net 3.3V: now also U3.2 (3V3); no longer U3.3 (3V3)
- net ESP19/D-: now also U3.13 (IO19); no longer U3.23 (IOA19)
- net ESP20/D+: now also U3.14 (IO20); no longer U3.24 (IOA20)
- net ESP35/~{ALRT}: now also U3.28 (IO35); no longer U3.31 (IO35)
- net ESP45/Q_EN: now also U3.26 (IO45); no longer U3.41 (IO45)
- net ESP9/SCL: now also U3.17 (IO9); no longer U3.13 (IOA9)
- net ESP~{RST}: now also U3.3 (EN); no longer U3.45 (EN)
- net GND: now also U3.40 (GND), U3.41 (EPAD); no longer U3.2 (GND), U3.42 (GND), U3.43 (GND), U3.46 (GND), U3.47 (GND), U3.48 (GND), U3.49 (GND), U3.50 (GND), U3.51 (GND), U3.52 (GND), U3.53 (GND), U3.54 (GND), U3.55 (GND), U3.56 (GND), U3.57 (GND), U3.58 (GND), U3.59 (GND), U3.60 (GND), U3.61 (GND), U3.62 (GND), U3.63 (GND), U3.64 (GND), U3.65 (GND)
- net ESP10/SPI_CS0: now reaches U3.18 (IO10)
- net ESP13/SPI0_MISO: now reaches U3.21 (IO13)
- net ESP14/BAT_ADC: now reaches U3.22 (IO14)
- net ESP4/TOUCH4: now reaches U3.4 (IO4)
- net ESP5/TOUCH5: now reaches U3.5 (IO5)
- net ESP6/TOUCH6: now reaches U3.6 (IO6)
- net ESP7/TOUCH7: now reaches U3.7 (IO7)
- net ESP15/XTAL_32K_P: now reaches U3.8 (IO15)
- net ESP16/XTAL_32K_N: now reaches U3.9 (IO16)
- net XTAL_32K_N renamed ESP12/SPI0_SCK
- net XTAL_32K_P renamed ESP11/SPI0_MOSI
Other:
- moved on the sheet: C6, R8, SW2

Commit message: temp
Parts:
- removed G1: qwiic_Logo, symbol SparkFun-Aesthetic:qwiic_Logo
- removed G2: SparkFun_Logo, symbol SparkFun-Aesthetic:SparkFun_Logo
- removed J1: USB_C_Receptacle, SparkFun-Connector:USB-C_16, symbol SparkFun-Connector:USB_C_Receptacle
- added C15: 1.0uF, Capacitor_SMD:C_0402_1005Metric, symbol SparkFun-Capacitor:1.0uF_0402_16V_10%
- added R3: 10k, Resistor_SMD:R_0402_1005Metric, symbol SparkFun-Resistor:10k_0402
- added SW1: C318884, EasyEDA_Lib:SW-SMD_4P-L5.1-W5.1-P3.70-LS6.5-TL_H1.5, symbol EasyEDA_Lib:TS-1187A-B-A-B
- added USB2: C2927038, EasyEDA_Lib:USB-C_SMD-TYPE-C-31-M-12, symbol EasyEDA_Lib:USB-TYPE-C-018
- C1: footprint SparkFun-Capacitor:C_0603_1608Metric -> Capacitor_SMD:C_0603_1608Metric
- C6, C7: footprint SparkFun-Capacitor:C_0402_1005Metric -> Capacitor_SMD:C_0402_1005Metric
- R10, R11, R13, R8: footprint SparkFun-Resistor:R_0402_1005Metric -> Resistor_SMD:R_0402_1005Metric
- SW2: value SMD_4.6x2.8mm_h2.5mm -> C318884; footprint SparkFun-Switch:Push_SMD_4.6x2.8mm_h2.5mm -> EasyEDA_Lib:SW-SMD_4P-L5.1-W5.1-P3.70-LS6.5-TL_H1.5; symbol SparkFun-Switch:SPST_Push_SMD_4.6x2.8mm_h2.5mm -> EasyEDA_Lib:TS-1187A-B-A-B; LCSC Part Name (none) -> 5.1*5.1*1.5mm 立贴 轻触开关; Manufacturer (none) -> XKB Connection(中国星坤); Manufacturer Part (none) -> TS-1187A-B-A-B; PROD_ID SWCH-15606 -> C318884; Supplier (none) -> LCSC; Supplier Part (none) -> C318884
- U2: value DT1042-04SO -> C85364; footprint SparkFun-Semiconductor-Standard:SOT23-6 -> EasyEDA_Lib:SOT-23-6_L2.9-W1.6-P0.95-LS2.9-BL; symbol SparkFun-DiscreteSemi:D_TVS_ESD_USB -> EasyEDA_Lib:SRV05-4A_C20615829; LCSC Part Name (none) -> 丝印:V05 单向ESD 5V截止 峰值浪涌电流：4A@8/20us; Manufacturer (none) -> R+O(宏嘉诚); Manufacturer Part (none) -> C85364; Supplier (none) -> LCSC; Supplier Part (none) -> C85364
- U3, U9: now not fitted
- U6: footprint SparkFun-Semiconductor-Standard:SOT23-5 -> Package_TO_SOT_SMD:SOT-23-5
Connections:
- net 3.3V: now also R3.1
- net ESP19/D-: now also USB2.A7 (DN1), USB2.B7 (DN2)
- net ESP20/D+: now also USB2.A6 (DP1), USB2.B6 (DP2)
- net ESP~{RST}: now also SW2.2 (B)
- net GND: now also SW2.3 (C), SW2.4 (D), C15.2, SW1.3 (C), SW1.4 (D), USB2.0 (SH), USB2.1 (SH), USB2.2 (SH), USB2.3 (SH), USB2.A1 (GND), USB2.A12 (GND), USB2.B1 (GND), USB2.B12 (GND); no longer SW2.2
- net VUSB: now also USB2.A4 (VBUS), USB2.A9 (VBUS), USB2.B4 (VBUS), USB2.B9 (VBUS)
- net at R11.1: now also USB2.A5 (CC1)
- net at R10.2: now also USB2.B5 (CC2)
- net ESP0/BOOT: now reaches U3.27 (IO0)
- net ESP0/BOOT: now also C15.1, R3.2, SW1.1 (A), SW1.2 (B)
Other:
- moved on the sheet: C6, R10, R11

Commit message: temp
Parts:
- added C16, C17: 1uF, Capacitor_SMD:C_0402_1005Metric, symbol SparkFun-Capacitor:2.2uF_0402_10V_10%
- added U8: ~, EasyEDA_Lib:SOT-353_L2.1-W1.3-P0.65-LS2.3-BL, symbol EasyEDA_Lib:ME6211C33R5G
Connections:
- net 3.3V: now also C17.1, U8.5 (VOUT)
- net GND: now also C16.2, C17.2, U8.2 (VSS)
- net VIN: now also C16.1, U8.1 (VIN), U8.3 (CE)
Other:
- note removed: "Differential Pair Calculation Copper Thickness (1oz): 1.4mil/0.035mm Board thickness: 1.6mm Dielectric thickness (layer 1 to 2): 7.9mil/0.2mm Er: 4.6 Trace Spacing: 6mil/0.1524mm Required Trace Width: 9mil/0.2286mm Source: Saturn PCB Toolkit"
- moved on the sheet: C10, C11, C13, R13, U6

Commit message: update schematic (hopefully final)
Parts:
- removed C10: 2.2uF, Capacitor_SMD:C_0402_1005Metric, symbol SparkFun-Capacitor:2.2uF_0402_10V_10%
- removed C11: 0.1uF, Capacitor_SMD:C_0402_1005Metric, symbol SparkFun-Capacitor:0.1uF_0402_6.3V_10%
- removed C13: 1.0uF, Capacitor_SMD:C_0402_1005Metric, symbol SparkFun-Capacitor:1.0uF_0402_16V_10%
- removed C16, C17: 1uF, Capacitor_SMD:C_0402_1005Metric, symbol SparkFun-Capacitor:2.2uF_0402_10V_10%
- removed G3: OSHW_Logo, SparkFun-Aesthetic:Creative_Commons_License, symbol SparkFun-Aesthetic:OSHW_Logo
- removed R13: 100k, Resistor_SMD:R_0402_1005Metric, symbol SparkFun-Resistor:100k_0402
- removed U6: RT9080-3.3, Package_TO_SOT_SMD:SOT-23-5, symbol SparkFun-Regulator:RT9080-3.3
- removed U9: ~, SparkFun-Aesthetic:Ordering_Instructions, symbol SparkFun-Aesthetic:Ordering_Instructions
- added C14, C3: 1uF, Capacitor_SMD:C_0402_1005Metric, symbol SparkFun-Capacitor:2.2uF_0402_10V_10%
- added D2: C8678, EasyEDA_Lib:SMA_L4.3-W2.6-LS5.2-RD, symbol EasyEDA_Lib:SS34_C8678
- added Q1: C10487, EasyEDA_Lib:SOT-23-3_L3.0-W1.7-P0.95-LS2.9-BR, symbol EasyEDA_Lib:SI2301CDS-T1-GE3
- added R6: 100k, Resistor_SMD:R_0402_1005Metric, symbol SparkFun-Resistor:100k_0402
- U3: now left out of the parts list
- U8: value ~ -> C235316
Connections:
- net 3.3V: now also C14.1
- net GND: now also C14.2, C3.2, R6.2
- net VUSB: now also D2.2 (A), Q1.1 (G), R6.1
- net ESP21/~{ALRT}: now reaches U3.23 (IO21)
- net ESP36/LED2: now reaches U3.29 (IO36)
- net ESP37/LED3: now reaches U3.30 (IO37)
- net ESP38/LED4: now reaches U3.31 (IO38)
- net ESP39/BUTTON1: now reaches U3.32 (IO39)
- net ESP40/BUTTON2: now reaches U3.33 (IO40)
- net ESP41/BUTTON3: now reaches U3.34 (IO41)
- net ESP42/BUTTON4: now reaches U3.35 (IO42)
- net ESP35/~{ALRT} renamed ESP35/LED1
- net VIN: no longer names the net of U8.1 (VIN), U8.3 (CE)
- net VIN: now also C3.1, D2.1 (K), Q1.2 (S)
- new net VBATT: Q1.3 (D)
Other:
- note added: "copy of https://kazulog.fun/en/dev-en/esp32-charge-by-lipo/#toc8"
- note removed: "Thing Plus Board Outline"
- moved on the sheet: C6, SW2, U8

Commit message: .
Connections:
- net ESP17/DC: now reaches U3.10 (IO17)
- net ESP2/RES: now reaches U3.38 (IO2)
- net ESP1/BUSY: now reaches U3.39 (IO1)
Changed lines of the file:
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@@
+		)
+	)
+	(global_label "ESP2{slash}RES"
+		(shape input)
+		(at 74.93 93.98 0)
+		(fields_autoplaced yes)
+		(effects
+			(font
+				(size 1.27 1.27)
+			)
+			(justify left)
+		)
+		(property "Intersheetrefs" "${INTERSHEET_REFS}"
+			(at 87.7122 93.98 0)
+			(effects
+				(font
+					(size 1.27 1.27)
+				)
+				(justify left)
+				(hide yes)
+			)
 		)
 	)
@@
 		)
 	)
+	(global_label "ESP17{slash}DC"
+		(shape input)
+		(at 74.93 132.08 0)
+		(fields_autoplaced yes)
+		(effects
+			(font
+				(size 1.27 1.27)
+			)
+			(justify left)
+		)
+		(property "Intersheetrefs" "${INTERSHEET_REFS}"
+			(at 87.8332 132.08 0)
+			(effects
+				(font
+					(size 1.27 1.27)
+				)
+				(justify left)
+				(hide yes)
+			)
+		)
+	)
 	(global_label "ESP~{RST}"
 		(shape input)
@@
 			(effects
 				(font
+					(size 1.27 1.27)
+				)
+				(justify left)
+				(hide yes)
+			)
+		)
+	)
+	(global_label "ESP1{slash}BUSY"
+		(shape input)
+		(at 74.93 91.44 0)
+		(fields_autoplaced yes)
+		(effects
+			(font
+				(size 1.27 1.27)
+			)
+			(justify left)
+		)
+		(property "Intersheetrefs" "${INTERSHEET_REFS}"
+			(at 88.9823 91.44 0)
+			(effects
+				(font

Commit message: 1st production version
Parts:
- removed R3: 10k, Resistor_SMD:R_0402_1005Metric, symbol SparkFun-Resistor:10k_0402
- removed ST1, ST3: Standoff, SparkFun-Hardware:Standoff, symbol SparkFun-Hardware:Standoff
- added H1, H2: MountingHole, MountingHole:MountingHole_6.4mm_M6_DIN965, symbol Mechanical:MountingHole
- added H3, H4, H5, H6: MountingHole, MountingHole:MountingHole_2.7mm_M2.5_ISO14580, symbol Mechanical:MountingHole
- U3: now in the parts list
- renumbered SW1 to BOOT1, SW2 to Reset1
