File: Hardware/riichi_compass.kicad_sch (KiCad schematic)
At the start: 24 parts, among them Q1 C10487, U2 C85364, U3 ESP32-S3-MINI, U8 C235316

Commit message: rename
Parts:
- U3: now fitted; now left out of the parts list
Other:
- sheet Peripherals: file SparkFun_Thing_Plus_ESP32-S3_Peripherals.kicad_sch -> riichi_compass_Peripherals.kicad_sch
- title: ESP32 Thing Plus ESP32-S3 -> riichi compass
Changed lines of the file:
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@@
 	(paper "USLetter")
 	(title_block
-		(title "ESP32 Thing Plus ESP32-S3")
-		(date "2023-07-28")
-		(rev "v10")
-		(comment 1 "Designed by: N.Seidle")
+		(title "riichi compass")
+		(date "2025-11-30")
+		(rev "v1")
 	)
 	(text "ESP32-S3"
@@
 		)
 		(instances
-			(project "SparkFun_Thing_Plus_ESP32-S3"
+			(project "riichi_compass"
 				(path "/e3dd3ae4-244d-4cba-9cca-5d2abf83f29a"
 					(reference "#PWR016")
@@
 		)
 		(instances
-			(project "SparkFun_Thing_Plus_ESP32-S3"
+			(project "riichi_compass"
 				(path "/e3dd3ae4-244d-4cba-9cca-5d2abf83f29a"
 					(reference "BOOT1")
@@
 		)
 		(instances
-			(project "SparkFun_Thing_Plus_ESP32-S3"
+			(project "riichi_compass"
 				(path "/e3dd3ae4-244d-4cba-9cca-5d2abf83f29a"
 					(reference "#PWR014")
@@
 		)
 		(instances
-			(project "SparkFun_Thing_Plus_ESP32-S3"
+			(project "riichi_compass"
 				(path "/e3dd3ae4-244d-4cba-9cca-5d2abf83f29a"
 					(reference "U8")
@@
 		)
 		(instances
-			(project "SparkFun_Thing_Plus_ESP32-S3"
+			(project "riichi_compass"
 				(path "/e3dd3ae4-244d-4cba-9cca-5d2abf83f29a"
 					(reference "C1")
@@
 		)
 		(instances
-			(project "SparkFun_Thing_Plus_ESP32-S3"
+			(project "riichi_compass"
 				(path "/e3dd3ae4-244d-4cba-9cca-5d2abf83f29a"
 					(reference "#PWR0101")
@@
 		)
 		(instances
-			(project "SparkFun_Thing_Plus_ESP32-S3"
+			(project "riichi_compass"
 				(path "/e3dd3ae4-244d-4cba-9cca-5d2abf83f29a"
 					(reference "D2")
@@
 				)
 			)
-			(project "SparkFun_Thing_Plus_ESP32-S3"
+			(project "riichi_compass"
 				(path "/e3dd3ae4-244d-4cba-9cca-5d2abf83f29a"
 					(reference "#PWR0115")
@@
 		)
 		(instances
-			(project "SparkFun_Thing_Plus_ESP32-S3"
+			(project "riichi_compass"
 				(path "/e3dd3ae4-244d-4cba-9cca-5d2abf83f29a"
 					(reference "#PWR017")
@@
 		)
 		(instances
-			(project "SparkFun_Thing_Plus_ESP32-S3"
+			(project "riichi_compass"
 				(path "/e3dd3ae4-244d-4cba-9cca-5d2abf83f29a"
 					(reference "H5")
@@
 		)
 		(instances
-			(project "SparkFun_Thing_Plus_ESP32-S3"
+			(project "riichi_compass"
 				(path "/e3dd3ae4-244d-4cba-9cca-5d2abf83f29a"
 					(reference "Q1")
@@
 				)
 			)
-			(project "SparkFun_Thing_Plus_ESP32-S3"
+			(project "riichi_compass"
 				(path "/e3dd3ae4-244d-4cba-9cca-5d2abf83f29a"
 					(reference "Reset1")
@@
 		)
 		(instances
-			(project "SparkFun_Thing_Plus_ESP32-S3"
+			(project "riichi_compass"
 				(path "/e3dd3ae4-244d-4cba-9cca-5d2abf83f29a"
 					(reference "R11")
@@
 		)
 		(instances
-			(project "SparkFun_Thing_Plus_ESP32-S3"
+			(project "riichi_compass"
 				(path "/e3dd3ae4-244d-4cba-9cca-5d2abf83f29a"
 					(reference "R6")
@@
 				)
 			)
-			(project "SparkFun_Thing_Plus_ESP32-S3"
+			(project "riichi_compass"
 				(path "/e3dd3ae4-244d-4cba-9cca-5d2abf83f29a"
 					(reference "C6")
@@
 				)
 			)
-			(project "SparkFun_Thing_Plus_ESP32-S3"
+			(project "riichi_compass"
 				(path "/e3dd3ae4-244d-4cba-9cca-5d2abf83f29a"
 					(reference "#PWR0120")
@@
 				)
 			)
-			(project "SparkFun_Thing_Plus_ESP32-S3"
+			(project "riichi_compass"
 				(path "/e3dd3ae4-244d-4cba-9cca-5d2abf83f29a"
 					(reference "R8")
@@
 		)
 		(instances
-			(project "SparkFun_Thing_Plus_ESP32-S3"
+			(project "riichi_compass"
 				(path "/e3dd3ae4-244d-4cba-9cca-5d2abf83f29a"
 					(reference "#PWR09")
@@
 				)
 			)
-			(project "SparkFun_Thing_Plus_ESP32-S3"
+			(project "riichi_compass"
 				(path "/e3dd3ae4-244d-4cba-9cca-5d2abf83f29a"
 					(reference "#PWR0121")
@@
 		)
 		(instances
-			(project "SparkFun_Thing_Plus_ESP32-S3"
+			(project "riichi_compass"
 				(path "/e3dd3ae4-244d-4cba-9cca-5d2abf83f29a"
 					(reference "U2")
@@
 		)
 		(instances
-			(project "SparkFun_Thing_Plus_ESP32-S3"
+			(project "riichi_compass"
 				(path "/e3dd3ae4-244d-4cba-9cca-5d2abf83f29a"
 					(reference "#PWR019")
@@
 		)
 		(instances
-			(project "SparkFun_Thing_Plus_ESP32-S3"
+			(project "riichi_compass"
 				(path "/e3dd3ae4-244d-4cba-9cca-5d2abf83f29a"
 					(reference "H2")
@@
 		)
 		(instances
-			(project "SparkFun_Thing_Plus_ESP32-S3"
+			(project "riichi_compass"
 				(path "/e3dd3ae4-244d-4cba-9cca-5d2abf83f29a"
 					(reference "C7")
@@
 		)
 		(instances
-			(project "SparkFun_Thing_Plus_ESP32-S3"
+			(project "riichi_compass"
 				(path "/e3dd3ae4-244d-4cba-9cca-5d2abf83f29a"
 					(reference "C14")
@@
 		)
 		(instances
-			(project "SparkFun_Thing_Plus_ESP32-S3"
+			(project "riichi_compass"
 				(path "/e3dd3ae4-244d-4cba-9cca-5d2abf83f29a"
 					(reference "#PWR04")
@@
 		)
 		(instances
-			(project "SparkFun_Thing_Plus_ESP32-S3"
+			(project "riichi_compass"
 				(path "/e3dd3ae4-244d-4cba-9cca-5d2abf83f29a"
 					(reference "H6")
@@
 		)
 		(instances
-			(project "SparkFun_Thing_Plus_ESP32-S3"
+			(project "riichi_compass"
 				(path "/e3dd3ae4-244d-4cba-9cca-5d2abf83f29a"
 					(reference "#PWR010")
@@
 				)
 			)
-			(project "SparkFun_Thing_Plus_ESP32-S3"
+			(project "riichi_compass"
 				(path "/e3dd3ae4-244d-4cba-9cca-5d2abf83f29a"
 					(reference "#PWR0116")
@@
 		)
 		(instances
-			(project "SparkFun_Thing_Plus_ESP32-S3"
+			(project "riichi_compass"
 				(path "/e3dd3ae4-244d-4cba-9cca-5d2abf83f29a"
 					(reference "#PWR012")
@@
 		)
 		(instances
-			(project "SparkFun_Thing_Plus_ESP32-S3"
+			(project "riichi_compass"
 				(path "/e3dd3ae4-244d-4cba-9cca-5d2abf83f29a"
 					(reference "#PWR011")
@@
 		)
 		(instances
-			(project "SparkFun_Thing_Plus_ESP32-S3"
+			(project "riichi_compass"
 				(path "/e3dd3ae4-244d-4cba-9cca-5d2abf83f29a"
 					(reference "H4")
@@
 		)
 		(instances
-			(project "SparkFun_Thing_Plus_ESP32-S3"
+			(project "riichi_compass"
 				(path "/e3dd3ae4-244d-4cba-9cca-5d2abf83f29a"
 					(reference "#PWR07")
@@
 		)
 		(instances
-			(project "SparkFun_Thing_Plus_ESP32-S3"
+			(project "riichi_compass"
 				(path "/e3dd3ae4-244d-4cba-9cca-5d2abf83f29a"
 					(reference "C3")
@@
 				)
 			)
-			(project "SparkFun_Thing_Plus_ESP32-S3"
+			(project "riichi_compass"
 				(path "/e3dd3ae4-244d-4cba-9cca-5d2abf83f29a"
 					(reference "#PWR0123")
@@
 				)
 			)
-			(project "SparkFun_Thing_Plus_ESP32-S3"
+			(project "riichi_compass"
 				(path "/e3dd3ae4-244d-4cba-9cca-5d2abf83f29a"
 					(reference "#PWR0112")
@@
 				)
 			)
-			(project "SparkFun_Thing_Plus_ESP32-S3"
+			(project "riichi_compass"
 				(path "/e3dd3ae4-244d-4cba-9cca-5d2abf83f29a"
 					(reference "#PWR0119")
@@
 		)
 		(instances
-			(project "SparkFun_Thing_Plus_ESP32-S3"
+			(project "riichi_compass"
 				(path "/e3dd3ae4-244d-4cba-9cca-5d2abf83f29a"
 					(reference "#PWR0105")
@@
 		)
 		(instances
-			(project "SparkFun_Thing_Plus_ESP32-S3"
+			(project "riichi_compass"
 				(path "/e3dd3ae4-244d-4cba-9cca-5d2abf83f29a"
 					(reference "R10")
@@
 		)
 		(instances
-			(project "SparkFun_Thing_Plus_ESP32-S3"
+			(project "riichi_compass"
 				(path "/e3dd3ae4-244d-4cba-9cca-5d2abf83f29a"
 					(reference "#PWR0102")
@@
 		)
 		(instances
-			(project "SparkFun_Thing_Plus_ESP32-S3"
+			(project "riichi_compass"
 				(path "/e3dd3ae4-244d-4cba-9cca-5d2abf83f29a"
 					(reference "#PWR018")
@@
 		(unit 1)
 		(exclude_from_sim no)
-		(in_bom yes)
+		(in_bom no)
 		(on_board yes)
-		(dnp yes)
+		(dnp no)
 		(fields_autoplaced yes)
 		(property "Reference" "U3"
@@
 		)
 		(instances
-			(project "SparkFun_Thing_Plus_ESP32-S3"
+			(project "riichi_compass"
 				(path "/e3dd3ae4-244d-4cba-9cca-5d2abf83f29a"
 					(reference "U3")
@@
 		)
 		(instances
-			(project "SparkFun_Thing_Plus_ESP32-S3"
+			(project "riichi_compass"
 				(path "/e3dd3ae4-244d-4cba-9cca-5d2abf83f29a"
 					(reference "C15")
@@
 			)
 		)
-		(property "Sheetfile" "SparkFun_Thing_Plus_ESP32-S3_Peripherals.kicad_sch"
+		(property "Sheetfile" "riichi_compass_Peripherals.kicad_sch"
 			(at 205.74 51.3846 0)
 			(effects
@@
 		)
 		(instances
-			(project "SparkFun_Thing_Plus_ESP32-S3"
+			(project "riichi_compass"
 				(path "/e3dd3ae4-244d-4cba-9cca-5d2abf83f29a"
 					(page "2")
